Commit message: [FIX]: fixed an issue with the agents colors
* updated core submodule to the HEAD (agent color fix at init)
* fixed custom viz to use colors just at init, not every update
* renamed nao meshes -> removed extra dots in names

File: res/templates/urdf/nao.urdf (robot description, URDF)
Before this commit: robot NaoH25V50, 79 links, 78 joints
Links:
- link Head: geometry collision mesh filename=nao_meshes/HeadPitch_0.stl scale=0.1 0.1 0.1; visual mesh filename=nao_meshes/HeadPitch_0.stl scale=0.1 0.1 0.1
- link LAnklePitch: geometry collision mesh filename=nao_meshes/LAnklePitch_0.stl scale=0.1 0.1 0.1; visual mesh filename=nao_meshes/LAnklePitch_0.stl scale=0.1 0.1 0.1
- link LBicep: geometry collision mesh filename=nao_meshes/LShoulderRoll_0.stl scale=0.1 0.1 0.1; visual mesh filename=nao_meshes/LShoulderRoll_0.stl scale=0.1 0.1 0.1
- link LFinger11_link: geometry collision mesh filename=nao_meshes/LFinger11_0.stl scale=0.1 0.1 0.1; visual mesh filename=nao_meshes/LFinger11_0.stl scale=0.1 0.1 0.1
- link LFinger12_link: geometry collision mesh filename=nao_meshes/LFinger12_0.stl scale=0.1 0.1 0.1; visual mesh filename=nao_meshes/LFinger12_0.stl scale=0.1 0.1 0.1
- link LFinger13_link: geometry collision mesh filename=nao_meshes/LFinger13_0.stl scale=0.1 0.1 0.1; visual mesh filename=nao_meshes/LFinger13_0.stl scale=0.1 0.1 0.1
- link LFinger21_link: geometry collision mesh filename=nao_meshes/LFinger21_0.stl scale=0.1 0.1 0.1; visual mesh filename=nao_meshes/LFinger21_0.stl scale=0.1 0.1 0.1
- link LFinger22_link: geometry collision mesh filename=nao_meshes/LFinger22_0.stl scale=0.1 0.1 0.1; visual mesh filename=nao_meshes/LFinger22_0.stl scale=0.1 0.1 0.1
- link LFinger23_link: geometry collision mesh filename=nao_meshes/LFinger23_0.stl scale=0.1 0.1 0.1; visual mesh filename=nao_meshes/LFinger23_0.stl scale=0.1 0.1 0.1
- link LForeArm: geometry collision mesh filename=nao_meshes/LElbowRoll_0.stl scale=0.1 0.1 0.1; visual mesh filename=nao_meshes/LElbowRoll_0.stl scale=0.1 0.1 0.1
- link LHip: geometry collision mesh filename=nao_meshes/LHipRoll_0.stl scale=0.1 0.1 0.1; visual mesh filename=nao_meshes/LHipRoll_0.stl scale=0.1 0.1 0.1
- link LPelvis: geometry collision mesh filename=nao_meshes/LHipYawPitch_0.stl scale=0.1 0.1 0.1; visual mesh filename=nao_meshes/LHipYawPitch_0.stl scale=0.1 0.1 0.1
- link LShoulder: geometry collision mesh filename=nao_meshes/LShoulderPitch_0.stl scale=0.1 0.1 0.1; visual mesh filename=nao_meshes/LShoulderPitch_0.stl scale=0.1 0.1 0.1
- link LThigh: geometry collision mesh filename=nao_meshes/LHipPitch_0.stl scale=0.1 0.1 0.1; visual mesh filename=nao_meshes/LHipPitch_0.stl scale=0.1 0.1 0.1
- link LThumb1_link: geometry collision mesh filename=nao_meshes/LThumb1_0.stl scale=0.1 0.1 0.1; visual mesh filename=nao_meshes/LThumb1_0.stl scale=0.1 0.1 0.1
- link LThumb2_link: geometry collision mesh filename=nao_meshes/LThumb2_0.stl scale=0.1 0.1 0.1; visual mesh filename=nao_meshes/LThumb2_0.stl scale=0.1 0.1 0.1
- link LTibia: geometry collision mesh filename=nao_meshes/LKneePitch_0.stl scale=0.1 0.1 0.1; visual mesh filename=nao_meshes/LKneePitch_0.stl scale=0.1 0.1 0.1
- link Neck: geometry collision mesh filename=nao_meshes/HeadYaw_0.stl scale=0.1 0.1 0.1; visual mesh filename=nao_meshes/HeadYaw_0.stl scale=0.1 0.1 0.1
- link RAnklePitch: geometry collision mesh filename=nao_meshes/RAnklePitch_0.stl scale=0.1 0.1 0.1; visual mesh filename=nao_meshes/RAnklePitch_0.stl scale=0.1 0.1 0.1
- link RBicep: geometry collision mesh filename=nao_meshes/RShoulderRoll_0.stl scale=0.1 0.1 0.1; visual mesh filename=nao_meshes/RShoulderRoll_0.stl scale=0.1 0.1 0.1
- link RFinger11_link: geometry collision mesh filename=nao_meshes/RFinger11_0.stl scale=0.1 0.1 0.1; visual mesh filename=nao_meshes/RFinger11_0.stl scale=0.1 0.1 0.1
- link RFinger12_link: geometry collision mesh filename=nao_meshes/RFinger12_0.stl scale=0.1 0.1 0.1; visual mesh filename=nao_meshes/RFinger12_0.stl scale=0.1 0.1 0.1
- link RFinger13_link: geometry collision mesh filename=nao_meshes/RFinger13_0.stl scale=0.1 0.1 0.1; visual mesh filename=nao_meshes/RFinger13_0.stl scale=0.1 0.1 0.1
- link RFinger21_link: geometry collision mesh filename=nao_meshes/RFinger21_0.stl scale=0.1 0.1 0.1; visual mesh filename=nao_meshes/RFinger21_0.stl scale=0.1 0.1 0.1
- link RFinger22_link: geometry collision mesh filename=nao_meshes/RFinger22_0.stl scale=0.1 0.1 0.1; visual mesh filename=nao_meshes/RFinger22_0.stl scale=0.1 0.1 0.1
- link RFinger23_link: geometry collision mesh filename=nao_meshes/RFinger23_0.stl scale=0.1 0.1 0.1; visual mesh filename=nao_meshes/RFinger23_0.stl scale=0.1 0.1 0.1
- link RForeArm: geometry collision mesh filename=nao_meshes/RElbowRoll_0.stl scale=0.1 0.1 0.1; visual mesh filename=nao_meshes/RElbowRoll_0.stl scale=0.1 0.1 0.1
- link RHip: geometry collision mesh filename=nao_meshes/RHipRoll_0.stl scale=0.1 0.1 0.1; visual mesh filename=nao_meshes/RHipRoll_0.stl scale=0.1 0.1 0.1
- link RPelvis: geometry collision mesh filename=nao_meshes/RHipYawPitch_0.stl scale=0.1 0.1 0.1; visual mesh filename=nao_meshes/RHipYawPitch_0.stl scale=0.1 0.1 0.1
- link RShoulder: geometry collision mesh filename=nao_meshes/RShoulderPitch_0.stl scale=0.1 0.1 0.1; visual mesh filename=nao_meshes/RShoulderPitch_0.stl scale=0.1 0.1 0.1
- link RThigh: geometry collision mesh filename=nao_meshes/RHipPitch_0.stl scale=0.1 0.1 0.1; visual mesh filename=nao_meshes/RHipPitch_0.stl scale=0.1 0.1 0.1
- link RThumb1_link: geometry collision mesh filename=nao_meshes/RThumb1_0.stl scale=0.1 0.1 0.1; visual mesh filename=nao_meshes/RThumb1_0.stl scale=0.1 0.1 0.1
- link RThumb2_link: geometry collision mesh filename=nao_meshes/RThumb2_0.stl scale=0.1 0.1 0.1; visual mesh filename=nao_meshes/RThumb2_0.stl scale=0.1 0.1 0.1
- link RTibia: geometry collision mesh filename=nao_meshes/RKneePitch_0.stl scale=0.1 0.1 0.1; visual mesh filename=nao_meshes/RKneePitch_0.stl scale=0.1 0.1 0.1
- link l_ankle: geometry collision mesh filename=nao_meshes/LAnkleRoll_0.stl scale=0.1 0.1 0.1; visual mesh filename=nao_meshes/LAnkleRoll_0.stl scale=0.1 0.1 0.1
- link l_wrist: geometry collision mesh filename=nao_meshes/LWristYaw_0.stl scale=0.1 0.1 0.1; visual mesh filename=nao_meshes/LWristYaw_0.stl scale=0.1 0.1 0.1
- link r_ankle: geometry collision mesh filename=nao_meshes/RAnkleRoll_0.stl scale=0.1 0.1 0.1; visual mesh filename=nao_meshes/RAnkleRoll_0.stl scale=0.1 0.1 0.1
- link r_wrist: geometry collision mesh filename=nao_meshes/RWristYaw_0.stl scale=0.1 0.1 0.1; visual mesh filename=nao_meshes/RWristYaw_0.stl scale=0.1 0.1 0.1
- link torso: geometry collision mesh filename=nao_meshes/Torso_0.stl scale=0.1 0.1 0.1; visual mesh filename=nao_meshes/Torso_0.stl scale=0.1 0.1 0.1
